Commit message: Added SLAM saving and updated launch accordingly

File: src/basic_gazebo_robot/urdf/my_robot.urdf (robot description, URDF)
Before this commit: robot my_robot, 4 links, 3 joints
Links:
- added link caster_link, mass 0.15; collision sphere radius=0.04; visual sphere radius=0.04
- link lidar_link: geometry collision cylinder length=0.08 radius=0.06; visual cylinder length=0.08 radius=0.06
Joints:
- added joint caster_joint: type fixed, parent base_link, child caster_link, origin xyz=0.25 0 0.06 rpy=0 0 0
- joint left_wheel_joint: origin xyz=0 0.23 0.1 rpy=0 0 0 -> xyz=-0.15 0.225 0.10 rpy=0 0 0
- joint lidar_joint: origin xyz=0 0 0.35 rpy=0 0 0 -> xyz=0 0 0.45 rpy=0 0 0
- joint right_wheel_joint: origin xyz=0 -0.23 0.1 rpy=0 0 0 -> xyz=-0.15 -0.225 0.10 rpy=0 0 0
